Commit message: Updated friction parameters

File: dyret_description/urdf/joints/foot.urdf.xacro (robot description, xacro)
@@ -79,11 +79,11 @@
 			</link>
 			<gazebo reference="${name}_foot_cyl2">
-				<mu1>0.5</mu1>
-				<mu2>0.5</mu2>
+				<mu1>0.7</mu1>
+				<mu2>0.7</mu2>
 				<kp>100000.0</kp>
 				<kd>1.0</kd>
 				<fdir1> 0.0 0.0 0.0 </fdir1>
 				<maxVel>0.001</maxVel>
-				<minDepth>0.001</minDepth>
+				<minDepth>0.000</minDepth>
 			</gazebo>
 			<joint name="${name}_foot_cyl_fixed" type="fixed">
@@ -110,14 +110,14 @@
 				<parent link="${name}_foot_cyl2" />
 				<child link="${name}_foot_sph" />
-				<origin xyz="0 0 ${-0.00975/2 - 0.0126/2 + 0.0101/2}" />
+				<origin xyz="0 0 -0.0063" />
 			</joint>
 			<gazebo reference="${name}_foot_sph">
-				<mu1>0.5</mu1>
-				<mu2>0.5</mu2>
+				<mu1>0.7</mu1>
+				<mu2>0.7</mu2>
 				<kp>100000.0</kp>
 				<kd>1.0</kd>
 				<fdir1> 0.0 0.0 0.0 </fdir1>
 				<maxVel>0.001</maxVel>
-				<minDepth>0.001</minDepth>
+				<minDepth>0.000</minDepth>
 				<material>Gazebo/Black</material>
 				<sensor name="${name}_bumper" type="contact">
