Commit message: Updated to new contact sensor build

File: dyret_description/urdf/dyret.xacro (robot description, xacro)
@@ -13,6 +13,6 @@
 			<updateRate>50</updateRate>
 			<pid>20000.0 0.0 100.0</pid>
-			<pid type="mx64">1000.0 0.5 1.0</pid>
-			<pid type="mx106">1000.0 0.5 1.0</pid>
+			<pid type="mx64">128.0 10.0 0.0</pid>
+			<pid type="mx106">128.0 10.0 0.0</pid>
 		</plugin>
 	</gazebo>

File: dyret_description/urdf/joints/foot.urdf.xacro (robot description, xacro)
@@ -3,4 +3,8 @@
 	<xacro:include filename="$(find dyret_description)/urdf/inertias.urdf.xacro" />
 	<xacro:macro name="foot" params="name">
+		<!-- The foot cylinder should always be included
+		     since the collision it represents is a stand-in
+		     for the larger 3D printed part below the extension
+		     leg (NOTE: it is a bit smaller, but should be large enough)-->
 		<link name="${name}_foot_cyl">
 			<collision>
@@ -12,35 +16,112 @@
 				radius="0.014"/>
 		</link>
-		<link name="${name}_foot_sph">
-			<visual>
-				<geometry>
-					<sphere radius="0.0142" />
-				</geometry>
-			</visual>
-			<collision>
-				<geometry>
-					<sphere radius="0.0142" />
-				</geometry>
-			</collision>
-			<xacro:box_inertia mass="0.018" height="0.0142"
-				width="0.0142" length="0.0142" />
-		</link>
-		<joint name="${name}_foot_fixed" type="fixed">
-			<parent link="${name}_foot_cyl" />
-			<child link="${name}_foot_sph" />
-			<origin xyz="0 0 ${-0.0355/2 + 0.00195}" />
-		</joint>
-		<xacro:if value="$(arg contact_enabled)">
+		<!-- Note that the foot cylinder is 3D printed and quite
+		     slippery, small values here should aid in avoiding
+		     behavior utilizing the cylinder to walk -->
+		<gazebo reference="${name}_foot_cyl">
+			<mu1>0.7</mu1>
+			<mu2>0.7</mu2>
+			<kp>100000.0</kp>
+			<kd>1.0</kd>
+			<maxVel>0.001</maxVel>
+			<minDepth>0.001</minDepth>
+		</gazebo>
+		<!-- If contact is not enabled we model the foot as a simple sphere
+		     with high friction parameters -->
+		<xacro:unless value="$(arg contact_enabled)">
+			<link name="${name}_foot_sph">
+				<visual>
+					<geometry>
+						<sphere radius="0.0142" />
+					</geometry>
+				</visual>
+				<collision>
+					<geometry>
+						<sphere radius="0.0142" />
+					</geometry>
+				</collision>
+				<xacro:box_inertia mass="0.018" height="0.0142"
+					width="0.0142" length="0.0142" />
+			</link>
+			<joint name="${name}_foot_fixed" type="fixed">
+				<parent link="${name}_foot_cyl" />
+				<child link="${name}_foot_sph" />
+				<origin xyz="0 0 ${-0.0355/2 + 0.00195}" />
+			</joint>
 			<gazebo reference="${name}_foot_sph">
-				<kp>1000000.0</kp>
-				<kd>100.0</kd>
+				<!-- 1.5 is very high friction -->
 				<mu1>1.5</mu1>
 				<mu2>1.5</mu2>
-				<maxVel>1.0</maxVel>
-				<minDepth>0.0</minDepth>
+				<kp>100000.0</kp>
+				<kd>1.0</kd>
+				<maxVel>0.001</maxVel>
+				<minDepth>0.001</minDepth>
+			</gazebo>
+		</xacro:unless>
+		<!-- The contact sensor is a bit smaller than the regular foot
+		     so we build it a bit down to avoid simulation being able
+		     to extend it sensor range -->
+		<xacro:if value="$(arg contact_enabled)">
+			<!-- Smaller cylinder: -->
+			<link name="${name}_foot_cyl2">
+				<collision>
+					<geometry>
+						<cylinder radius="0.011" length="0.0126" />
+					</geometry>
+				</collision>
+				<visual>
+					<geometry>
+						<cylinder radius="0.011" length="0.0126" />
+					</geometry>
+				</visual>
+				<xacro:cylinder_inertia mass="0.009" height="0.0126"
+					radius="0.011"/>
+			</link>
+			<gazebo reference="${name}_foot_cyl2">
+				<mu1>0.5</mu1>
+				<mu2>0.5</mu2>
+				<kp>100000.0</kp>
+				<kd>1.0</kd>
+				<fdir1> 0.0 0.0 0.0 </fdir1>
+				<maxVel>0.001</maxVel>
+				<minDepth>0.001</minDepth>
+			</gazebo>
+			<joint name="${name}_foot_cyl_fixed" type="fixed">
+				<parent link="${name}_foot_cyl" />
+				<child link="${name}_foot_cyl2" />
+				<origin xyz="0 0 ${-0.0355/2 - 0.0126/2}" />
+			</joint>
+			<!-- Smaller sphere with sensor: -->
+			<link name="${name}_foot_sph">
+				<visual>
+					<geometry>
+						<sphere radius="0.01" />
+					</geometry>
+				</visual>
+				<collision>
+					<geometry>
+						<sphere radius="0.01" />
+					</geometry>
+				</collision>
+				<xacro:box_inertia mass="0.009" height="0.00975"
+					width="0.00975" length="0.00975" />
+			</link>
+			<joint name="${name}_foot_fixed" type="fixed">
+				<parent link="${name}_foot_cyl2" />
+				<child link="${name}_foot_sph" />
+				<origin xyz="0 0 ${-0.00975/2 - 0.0126/2 + 0.0101/2}" />
+			</joint>
+			<gazebo reference="${name}_foot_sph">
+				<mu1>0.5</mu1>
+				<mu2>0.5</mu2>
+				<kp>100000.0</kp>
+				<kd>1.0</kd>
+				<fdir1> 0.0 0.0 0.0 </fdir1>
+				<maxVel>0.001</maxVel>
+				<minDepth>0.001</minDepth>
 				<material>Gazebo/Black</material>
 				<sensor name="${name}_bumper" type="contact">
 					<contact>
-						<collision>${name}_ext1_outer_fixed_joint_lump__${name}_foot_sph_collision_2</collision>
+						<collision>${name}_ext1_outer_fixed_joint_lump__${name}_foot_sph_collision_3</collision>
 					</contact>
 					<plugin name="${name}_gazebo_ros_bumper_controller"
@@ -54,21 +135,5 @@
 		</xacro:if>
 		<xacro:unless value="$(arg contact_enabled)">
-			<gazebo reference="${name}_foot_sph">
-				<kp>1000000.0</kp>
-				<kd>100.0</kd>
-				<mu1>1.5</mu1>
-				<mu2>1.5</mu2>
-				<maxVel>1.0</maxVel>
-				<minDepth>0.0</minDepth>
-			</gazebo>
 		</xacro:unless>
-		<gazebo reference="${name}_foot_cyl">
-			<kp>1000000.0</kp>
-			<kd>100.0</kd>
-			<mu1>1.5</mu1>
-			<mu2>1.5</mu2>
-			<maxVel>1.0</maxVel>
-			<minDepth>0.0</minDepth>
-		</gazebo>
 	</xacro:macro>
 </robot>

File: dyret_description/urdf/joints/mx106.urdf.xacro (robot description, xacro)
@@ -114,12 +114,10 @@
 			<limit
 				lower="-1.57" upper="1.57"
-				effort="10.0" velocity="5.76" />
-			<dynamics friction="0.1" damping="0.0952" />
+				effort="30.0" velocity="5.76" />
+			<!--<dynamics friction="0.1" damping="0.0952" />-->
+			<dynamics friction="0.3" damping="3.0" />
 		</joint>
 		<gazebo reference="${name}">
 			<implicitSpringDamper>1</implicitSpringDamper>
-			<stopKd value="100000000.0" />
-			<stopKp value="100000000.0" />
-			<fudgeFactor value="0.5" />
 		</gazebo>
 	</xacro:macro>
@@ -133,12 +131,10 @@
 			<limit
 				lower="-1.57" upper="1.57"
-				effort="10.0" velocity="5.76" />
-			<dynamics friction="0.1" damping="0.0952" />
+				effort="30.0" velocity="5.76" />
+			<!--<dynamics friction="0.1" damping="0.0952" />-->
+			<dynamics friction="0.3" damping="3.0" />
 		</joint>
 		<gazebo reference="${name}">
 			<implicitSpringDamper>1</implicitSpringDamper>
-			<stopKd value="100000000.0" />
-			<stopKp value="100000000.0" />
-			<fudgeFactor value="0.5" />
 		</gazebo>
 	</xacro:macro>

File: dyret_description/urdf/joints/mx64at.urdf.xacro (robot description, xacro)
@@ -69,12 +69,10 @@
 			<limit
 				lower="-1.57" upper="1.57"
-				effort="6.0" velocity="6.597" />
-			<dynamics friction="0.1" damping="0.0952" />
+				effort="30.0" velocity="6.597" />
+			<!--<dynamics friction="0.1" damping="0.0952" />-->
+			<dynamics friction="0.3" damping="3.0" />
 		</joint>
 		<gazebo reference="${name}">
 			<implicitSpringDamper>1</implicitSpringDamper>
-			<stopKd value="100000000.0" />
-			<stopKp value="100000000.0" />
-			<fudgeFactor value="0.5" />
 		</gazebo>
 	</xacro:macro>

Commit message: Fixed error in PID setting and updated some PID values

File: dyret_description/urdf/dyret.xacro (robot description, xacro)
@@ -12,5 +12,5 @@
 		<plugin name="controller" filename="libdyret_gazebo_plugin.so">
 			<updateRate>50</updateRate>
-			<pid>20000.0 0.0 100.0</pid>
+			<pid>2000.0 200.0 0.0</pid>
 			<pid type="mx64">128.0 10.0 0.0</pid>
 			<pid type="mx106">128.0 10.0 0.0</pid>

File: dyret_description/urdf/joints/large_extend.urdf.xacro (robot description, xacro)
@@ -60,6 +60,6 @@
 			<limit
 				lower="-0.100" upper="0.0"
-				effort="100.0" velocity="0.00045" />
-			<dynamics damping="1.0" friction="70" />
+				effort="10000.0" velocity="0.00045" />
+			<dynamics damping="50.0"/>
 		</joint>
 		<gazebo reference="${name}">

File: dyret_description/urdf/joints/small_extend.urdf.xacro (robot description, xacro)
@@ -58,6 +58,6 @@
 			<limit
 				lower="-0.025" upper="0.0"
-				effort="100.0" velocity="0.00045" />
-			<dynamics damping="1.0" friction="80" />
+				effort="10000.0" velocity="0.00000045" />
+			<dynamics damping="50.0"/>
 		</joint>
 		<gazebo reference="${name}">
